Commit message: Improve Gazebo lidar simulation and wheel dynamics
- make the lidar merger follow the rotating joint and publish a 360 degree scan
- add cylindrical wheel collisions with friction tuning for better Gazebo contact
- introduce a custom Gazebo world with sensor plugins and boundary walls
- update launch, controller, and packaging files for the new simulation setup
- refresh the ROS helper script to rebuild and source the workspace before launching

File: src/lidarino_description/urdf/Lidarino.urdf (robot description, URDF)
Before this commit: robot Lidarino, 8 links, 7 joints
Links:
- link wheel_L: geometry collision cylinder length=0.025 radius=0.035; visual mesh filename=package://lidarino_description/urdf/meshes/wheel_L.stl scale=0.001 0.001 0.001
- link wheel_R: geometry collision cylinder length=0.025 radius=0.035; visual mesh filename=package://lidarino_description/urdf/meshes/wheel_R.stl scale=0.001 0.001 0.001
Joints:
- joint tof_1_joint: origin xyz=0.043 0.0 -0.031 rpy=0 0 0 -> xyz=0.044 0.0 -0.031 rpy=0 0 0
- joint tof_2_joint: origin xyz=2.6329906181668093e-18 0.043 -0.031 rpy=0 0 1.5707963267948966 -> xyz=2.694222958124177e-18 0.044 -0.031 rpy=0 0 1.5707963267948966
- joint tof_3_joint: origin xyz=-0.043 5.265981236333619e-18 -0.031 rpy=0 0 3.141592653589793 -> xyz=-0.044 5.388445916248354e-18 -0.031 rpy=0 0 3.141592653589793
- joint tof_4_joint: origin xyz=-7.898971854500428e-18 -0.043 -0.031 rpy=0 0 4.71238898038469 -> xyz=-8.08266887437253e-18 -0.044 -0.031 rpy=0 0 4.71238898038469

File: src/lidarino_description/urdf/Lidarino.urdf.xacro (robot description, xacro)
@@ -15,7 +15,8 @@
         </visual>
         <collision name="wheel_R_collision">
-            <origin xyz="1.1368683772161603e-15 1.3322676295501878e-17 0.0" rpy="-4.72621546065603e-16 -1.1102230246251568e-16 -2.7755575615628926e-17" />
+            <origin xyz="0 0 -0.017" rpy="0 0 0" />
             <geometry>
-                <mesh filename="${mesh_url}wheel_R.stl" scale="0.001 0.001 0.001" />
+                <cylinder radius="0.035" length="0.025" />
+                <!-- <mesh filename="${mesh_url}wheel_R.stl" scale="0.001 0.001 0.001" /> -->
             </geometry>
         </collision>
@@ -53,7 +54,8 @@
         </visual>
         <collision name="wheel_L_collision">
-            <origin xyz="1.1368683772161603e-15 1.1102230246251566e-17 0.0" rpy="-1.4649353258190343e-16 -1.2470396389907355e-32 -5.551115123125783e-17" />
+            <origin xyz="0 0 -0.017" rpy="0 0 0" />
             <geometry>
-                <mesh filename="${mesh_url}wheel_L.stl" scale="0.001 0.001 0.001" />
+                <cylinder radius="0.035" length="0.025" />
+                <!-- <mesh filename="${mesh_url}wheel_L.stl" scale="0.001 0.001 0.001" /> -->
             </geometry>
         </collision>
@@ -166,3 +168,15 @@
         </plugin>
     </gazebo>
+    <gazebo reference="wheel_R">
+        <mu1>1.0</mu1>
+        <mu2>1.0</mu2>
+        <kp>1000000.0</kp>
+        <kd>100.0</kd>
+    </gazebo>
+    <gazebo reference="wheel_L">
+        <mu1>1.0</mu1>
+        <mu2>1.0</mu2>
+        <kp>1000000.0</kp>
+        <kd>100.0</kd>
+    </gazebo>
 </robot>

Commit message: Add differential drive teleop and improve simulation stability
- add a diff drive controller so the robot can be driven from the keyboard and launched from ros_manager.py
- switch wheel collision geometry to spheres to reduce simulation drift
- retune mass and inertia values to better match the lighter 3D printed robot
- update Gazebo launch and controller configuration for the new drive setup

File: src/lidarino_description/urdf/Lidarino.urdf (robot description, URDF)
Before this commit: robot Lidarino, 8 links, 7 joints
Links:
- link base_link: mass 1.44483758348271 -> 0.23452271908044364
- link lidar: mass 0.4019930481298474 -> 0.05517921789897613
- link wheel_L: geometry collision sphere radius=0.035; visual mesh filename=package://lidarino_description/urdf/meshes/wheel_L.stl scale=0.001 0.001 0.001
- link wheel_R: geometry collision sphere radius=0.035; visual mesh filename=package://lidarino_description/urdf/meshes/wheel_R.stl scale=0.001 0.001 0.001
Joints:
- joint L_wheel_Revolute: axis 0.0 0.0 1.0 -> 0.0 0.0 -1.0; limit (none) -> effort=10.0 velocity=20.0
- joint R_wheel_Revolute: limit (none) -> effort=10.0 velocity=20.0

File: src/lidarino_description/urdf/Lidarino.urdf.xacro (robot description, xacro)
@@ -17,6 +17,5 @@
             <origin xyz="0 0 -0.017" rpy="0 0 0" />
             <geometry>
-                <cylinder radius="0.035" length="0.025" />
-                <!-- <mesh filename="${mesh_url}wheel_R.stl" scale="0.001 0.001 0.001" /> -->
+                <sphere radius="0.035" />
             </geometry>
         </collision>
@@ -25,6 +24,6 @@
         <inertial>
             <origin xyz="-0.003112056333080186 -2.296575824702822e-16 0.00763198155223819" rpy="0.0 0.0 0.0" />
-            <mass value="1.44483758348271" />
-            <inertia ixx="0.0025457615441212243" iyy="0.00441386927796519" izz="0.006647237489877395" ixy="6.620894401158822e-14" iyz="5.9584279388141974e-12" ixz="0.00017302389203673375" />
+            <mass value="0.23452271908044364" />
+            <inertia ixx="0.00044352479067893535" iyy="0.0006700968102651768" izz="0.001064913287950513" ixy="8.940708824769937e-15" iyz="3.5156320803171255e-12" ixz="3.3751097963762396e-05" />
         </inertial>
         <visual name="base_link_visual">
@@ -56,6 +55,5 @@
             <origin xyz="0 0 -0.017" rpy="0 0 0" />
             <geometry>
-                <cylinder radius="0.035" length="0.025" />
-                <!-- <mesh filename="${mesh_url}wheel_L.stl" scale="0.001 0.001 0.001" /> -->
+                <sphere radius="0.035" />
             </geometry>
         </collision>
@@ -64,6 +62,6 @@
         <inertial>
             <origin xyz="9.148285995408401e-10 -1.4055638260363446e-14 -0.018366241687653523" rpy="0.0 -0.0 0.0" />
-            <mass value="0.4019930481298474" />
-            <inertia ixx="0.0002920255957537354" iyy="0.0002920255955669725" izz="0.00046610883762024824" ixy="4.5174590427356237e-13" iyz="-5.303116405096e-16" ixz="1.832046775569751e-12" />
+            <mass value="0.05517921789897613" />
+            <inertia ixx="4.035574913846524e-05" iyy="4.035574911324637e-05" izz="6.456345828808408e-05" ixy="6.10000891607277e-14" iyz="-7.147133370998126e-17" ixz="2.3863745181318397e-13" />
         </inertial>
         <visual name="lidar_visual">
@@ -84,5 +82,6 @@
         <parent link="base_link" />
         <child link="wheel_L" />
-        <axis xyz="0.0 0.0 1.0" />
+        <axis xyz="0.0 0.0 -1.0" />
+        <limit effort="10.0" velocity="20.0" />
     </joint>
     <joint name="R_wheel_Revolute" type="continuous">
@@ -91,4 +90,5 @@
         <child link="wheel_R" />
         <axis xyz="0.0 0.0 1.0" />
+        <limit effort="10.0" velocity="20.0" />
     </joint>
     <joint name="lidar_Revolute" type="continuous">
@@ -157,8 +157,18 @@
         </joint>
         <joint name="R_wheel_Revolute">
+            <command_interface name="velocity">
+                <param name="min">-10</param>
+                <param name="max">10</param>
+            </command_interface>
             <state_interface name="position"/>
+            <state_interface name="velocity"/>
         </joint>
         <joint name="L_wheel_Revolute">
+            <command_interface name="velocity">
+                <param name="min">-10</param>
+                <param name="max">10</param>
+            </command_interface>
             <state_interface name="position"/>
+            <state_interface name="velocity"/>
         </joint>
     </ros2_control>
@@ -167,4 +177,8 @@
             <parameters>$(find lidarino_description)/config/controllers.yaml</parameters>
         </plugin>
+    </gazebo>
+    <gazebo reference="base_link">
+        <mu1>0.0</mu1>
+        <mu2>0.0</mu2>
     </gazebo>
     <gazebo reference="wheel_R">
