Commit message: Bug fix: Add fixed joint for caster - Added a fixed joint for the caster to ensure it is properly attached to the base link. - Updated the collision properties for the caster to prevent it from affecting the robot's movement. - Better approximated the mass and inertia properties of the camera for more accurate simulation.

File: src/lidarino_description/urdf/astra_camera.xacro (robot description, xacro)
@@ -17,5 +17,5 @@
             <inertial>
                 <mass value="0.3" />
-                <inertia ixx="0.0001" iyy="0.0001" izz="0.0001" ixy="0" iyz="0" ixz="0" />
+                <inertia ixx="0.000703" iyy="0.000063" izz="0.000721" ixy="0" iyz="0" ixz="0" />
             </inertial>
         </link>

File: src/lidarino_description/urdf/lidarino_core.xacro (robot description, xacro)
@@ -15,7 +15,27 @@
         </visual>
         <collision name="base_link_collision">
+            <origin xyz="0.0 0.0 0.015" rpy="0.0 0.0 0.0" />
+            <geometry>
+                <box size="0.2 0.12 0.03" />
+            </geometry>
+        </collision>
+    </link>
+    <link name="caster">
+        <inertial>
+            <origin xyz="0.0 0.0 0.0" rpy="0.0 0.0 0.0" />
+            <mass value="0.01" />
+            <inertia ixx="1e-6" iyy="1e-6" izz="1e-6" ixy="0" iyz="0" ixz="0" />
+        </inertial>
+        <visual name="caster_visual">
             <origin xyz="0.0 0.0 0.0" rpy="0.0 0.0 0.0" />
             <geometry>
-                <mesh filename="${mesh_url}base_link.stl" scale="0.001 0.001 0.001" />
+                <sphere radius="0.008" />
+            </geometry>
+            <material name="silver" />
+        </visual>
+        <collision name="caster_collision">
+            <origin xyz="0.0 0.0 0.0" rpy="0.0 0.0 0.0" />
+            <geometry>
+                <sphere radius="0.008" />
             </geometry>
         </collision>
@@ -101,3 +121,8 @@
         <axis xyz="0.0 0.0 1.0" />
     </joint>
+    <joint name="caster_fixed" type="fixed">
+        <origin xyz="0.052 0.0 -0.013" rpy="0.0 0.0 0.0" />
+        <parent link="base_link" />
+        <child link="caster" />
+    </joint>
 </robot>

File: src/lidarino_description/urdf/lidarino_gazebo.xacro (robot description, xacro)
@@ -7,4 +7,8 @@
     </gazebo>
     <gazebo reference="base_link">
+        <mu1>0.0</mu1>
+        <mu2>0.0</mu2>
+    </gazebo>
+    <gazebo reference="caster">
         <mu1>0.0</mu1>
         <mu2>0.0</mu2>

Commit message: BIG CHANGES IN THIS COMMIT: - Added support for Lidarino s2 (RPLIDAR S2) in the ROS 2 workspace (meshes, urdf, launch files). - Added possibility of choosing the Lidarino version in the ROS 2 manager, with Lidarino S2 as the default option. - Removed the option to activate the lidar in the ROS 2 manager, as it is not necessary for Lidarino S2. - Added launch files for SLAM and Navigation, which are now available in the ROS 2 manager. - Now gazebo.launch.py automatically launches the controller, SLAM, and Navigation for Lidarino S2. - Modified the display.launch.py file to just display the model in Rviz2 with right configurations defined in config/justRobot.rviz. - Added new world: apartment.world, selectable when launching Gazebo. - Added nav2_params.yaml for Navigation2 configuration. - Renamed the following files to indicate they are for Lidarino v1:   - controllers.yaml -> controllers_v1.yaml   - mapper_params_online_async.yaml -> mapper_params_v1.yaml   - lidarino_core.xacro -> lidarino_core_v1.xacro   - lidarino.urdf.xacro -> lidarino_v1.urdf.xacro - Added new files for Lidarino S2:   - controllers_s2.yaml   - mapper_params_s2.yaml   - lidarino_core_s2.xacro   - lidarino_s2.urdf.xacro   - rplidars2.xacro   - meshes/RPLIDARS2.stl   - meshes/base_link_s2.stl - Modified lidarino_ros2_control.xacro to support both Lidarino v1 and S2. - Modified lidarino_gazebo.xacro to support both Lidarino v1 and S2. - Added black color to the RPLIDAR S2 mesh in materials.xacro. - Now astra_camera.xacro uses the new mesh astra_camera.stl instead of the old one.

File: src/lidarino_description/urdf/astra_camera.xacro (robot description, xacro)
@@ -3,20 +3,22 @@
     <xacro:macro name="astra_camera" params="parent xyz rpy">
         <link name="astra_link">
-            <visual>
+            <inertial>
+                <origin xyz="0.021745856967737336 3.8230579211581216e-05 0.029303333814809707" rpy="0.0 0.0 0.0" />
+                <mass value="0.23334756462839484" />
+                <inertia ixx="0.00045538823905664865" iyy="7.785663760045297e-05" izz="0.00045460807011731756" ixy="1.841447020567419e-07" iyz="-4.2054876695014596e-08" ixz="9.205395041665818e-06" />
+            </inertial>
+            <visual name="astracamera_visual">
+                <origin xyz="0.0 0.0 0.0" rpy="0.0 0.0 0.0" />
                 <geometry>
-                    <box size="0.04 0.165 0.03" />
+                    <mesh filename="${mesh_url}astracamera.stl" scale="0.001 0.001 0.001" />
                 </geometry>
-                <material name="dark_grey">
-                </material>
+                <material name="dark_grey" />
             </visual>
-            <collision>
+            <collision name="astracamera_collision">
+                <origin xyz="0.0 0.0 0.0" rpy="0.0 0.0 0.0" />
                 <geometry>
-                    <box size="0.04 0.165 0.03" />
+                    <mesh filename="${mesh_url}astracamera.stl" scale="0.001 0.001 0.001" />
                 </geometry>
             </collision>
-            <inertial>
-                <mass value="0.3" />
-                <inertia ixx="0.000703" iyy="0.000063" izz="0.000721" ixy="0" iyz="0" ixz="0" />
-            </inertial>
         </link>
         <joint name="astra_joint" type="fixed">
@@ -29,11 +31,11 @@
             <parent link="astra_link" />
             <child link="astra_optical_frame" />
-            <origin xyz="0 0 0" rpy="-1.57079632679 0 -1.57079632679" />
+            <origin xyz="0 0 0.032" rpy="${rpy}" />
         </joint>
-        <gazebo reference="astra_link">
+        <gazebo reference="astra_optical_frame">
             <sensor type="rgbd_camera" name="astra_pro">
                 <topic>/astra/camera</topic>
                 <always_on>true</always_on>
-                <update_rate>30.0</update_rate>
+                <update_rate>5.0</update_rate>
                 <camera>
                     <horizontal_fov>1.047</horizontal_fov>

File: src/lidarino_description/urdf/lidarino_gazebo.xacro (robot description, xacro)
@@ -1,28 +1,31 @@
 <?xml version='1.0' encoding='utf-8'?>
 <robot xmlns:xacro="http://www.ros.org/wiki/xacro">
-    <gazebo>
-        <plugin filename="gz_ros2_control-system" name="gz_ros2_control::GazeboSimROS2ControlPlugin">
-            <parameters>$(find lidarino_description)/config/controllers.yaml</parameters>
-        </plugin>
-    </gazebo>
-    <gazebo reference="base_link">
-        <mu1>0.0</mu1>
-        <mu2>0.0</mu2>
-    </gazebo>
-    <gazebo reference="caster">
-        <mu1>0.0</mu1>
-        <mu2>0.0</mu2>
-    </gazebo>
-    <gazebo reference="wheel_R">
-        <mu1>1.0</mu1>
-        <mu2>1.0</mu2>
-        <kp>1000000.0</kp>
-        <kd>100.0</kd>
-    </gazebo>
-    <gazebo reference="wheel_L">
-        <mu1>1.0</mu1>
-        <mu2>1.0</mu2>
-        <kp>1000000.0</kp>
-        <kd>100.0</kd>
-    </gazebo>
+    <xacro:macro name="lidarino_gazebo" params="yaml_file">
+        <gazebo>
+            <plugin filename="gz_ros2_control-system" name="gz_ros2_control::GazeboSimROS2ControlPlugin">
+                <parameters>${yaml_file}</parameters>
+                <controller_manager_node_name>controller_manager</controller_manager_node_name>
+            </plugin>
+        </gazebo>
+        <gazebo reference="base_link">
+            <mu1>0.0</mu1>
+            <mu2>0.0</mu2>
+        </gazebo>
+        <gazebo reference="caster">
+            <mu1>0.0</mu1>
+            <mu2>0.0</mu2>
+        </gazebo>
+        <gazebo reference="wheel_R">
+            <mu1>1.0</mu1>
+            <mu2>1.0</mu2>
+            <kp>1000000.0</kp>
+            <kd>100.0</kd>
+        </gazebo>
+        <gazebo reference="wheel_L">
+            <mu1>1.0</mu1>
+            <mu2>1.0</mu2>
+            <kp>1000000.0</kp>
+            <kd>100.0</kd>
+        </gazebo>
+    </xacro:macro>
 </robot>

File: src/lidarino_description/urdf/lidarino_ros2_control.xacro (robot description, xacro)
@@ -1,32 +1,36 @@
 <?xml version='1.0' encoding='utf-8'?>
 <robot xmlns:xacro="http://www.ros.org/wiki/xacro">
-    <ros2_control name="GazeboSystem" type="system">
-        <hardware>
-            <plugin>gz_ros2_control/GazeboSimSystem</plugin>
-        </hardware>
-        <joint name="lidar_Revolute">
-            <command_interface name="velocity">
-                <param name="min">-100</param>
-                <param name="max">100</param>
-            </command_interface>
-            <state_interface name="position"/>
-            <state_interface name="velocity"/>
-        </joint>
-        <joint name="R_wheel_Revolute">
-            <command_interface name="velocity">
-                <param name="min">-10</param>
-                <param name="max">10</param>
-            </command_interface>
-            <state_interface name="position"/>
-            <state_interface name="velocity"/>
-        </joint>
-        <joint name="L_wheel_Revolute">
-            <command_interface name="velocity">
-                <param name="min">-10</param>
-                <param name="max">10</param>
-            </command_interface>
-            <state_interface name="position"/>
-            <state_interface name="velocity"/>
-        </joint>
-    </ros2_control>
+    <xacro:macro name="lidarino_ros2_control" params="use_lidar_control">
+        <ros2_control name="GazeboSystem" type="system">
+            <hardware>
+                <plugin>gz_ros2_control/GazeboSimSystem</plugin>
+            </hardware>
+            <xacro:if value="${use_lidar_control}">
+                <joint name="lidar_Revolute">
+                    <command_interface name="velocity">
+                        <param name="min">-100</param>
+                        <param name="max">100</param>
+                    </command_interface>
+                    <state_interface name="position"/>
+                    <state_interface name="velocity"/>
+                </joint>
+            </xacro:if>
+            <joint name="R_wheel_Revolute">
+                <command_interface name="velocity">
+                    <param name="min">-10</param>
+                    <param name="max">10</param>
+                </command_interface>
+                <state_interface name="position"/>
+                <state_interface name="velocity"/>
+            </joint>
+            <joint name="L_wheel_Revolute">
+                <command_interface name="velocity">
+                    <param name="min">-10</param>
+                    <param name="max">10</param>
+                </command_interface>
+                <state_interface name="position"/>
+                <state_interface name="velocity"/>
+            </joint>
+        </ros2_control>
+    </xacro:macro>
 </robot>

File: src/lidarino_description/urdf/lidarino_v1.urdf.xacro (robot description, xacro)
@@ -3,8 +3,11 @@
     <xacro:property name="mesh_url" value="package://lidarino_description/urdf/meshes/" />
     <xacro:include filename="materials.xacro" />
-    <xacro:include filename="lidarino_core.xacro" />
+    <xacro:include filename="lidarino_core_v1.xacro" />
     <xacro:include filename="tof_sensor.xacro" />
+    <xacro:arg name="yaml_file" default="$(find lidarino_description)/config/controllers_v1.yaml" />
     <xacro:include filename="lidarino_gazebo.xacro" />
     <xacro:include filename="lidarino_ros2_control.xacro" />
+    <xacro:lidarino_gazebo yaml_file="$(arg yaml_file)" />
+    <xacro:lidarino_ros2_control use_lidar_control="true" />
     <xacro:include filename="astra_camera.xacro" />
     <xacro:tof_sensor id="1" angle="0"          parent="lidar" />

File: src/lidarino_description/urdf/materials.xacro (robot description, xacro)
@@ -1,6 +1,9 @@
 <?xml version="1.0" encoding="utf-8"?>
 <robot xmlns:xacro="http://www.ros.org/wiki/xacro">
+    <material name="black">
+        <color rgba="0.1 0.1 0.1 1.0"/>
+    </material>
     <material name="dark_grey">
-        <color rgba="0.2 0.2 0.2 1.0"/>
+        <color rgba="0.25 0.25 0.25 1.0"/>
     </material>
     <material name="matte_orange">

Commit message: Autonomous exploration, Imu, EKF, optimization - Created file launch_sim.sh to launch the simulation with Gazebo and avoid ctrl-c problems - Added imu.xacro file to the lidarino_description package - Added ekf.yaml file to the lidarino_description package - Implemented imu and ekf to have better localization and navigation - Added explore.yaml file to the lidarino_description package - Added option to ros_manager.py to launch the exploration node - Simplified collisions of Astra Camera and RPLidarS2 for optimization purposes - Added lower objects in the apartment world to check if astra camera can detect them and avoid collisions that lidar cannot detect

File: src/lidarino_description/urdf/astra_camera.xacro (robot description, xacro)
@@ -16,7 +16,8 @@
             </visual>
             <collision name="astracamera_collision">
-                <origin xyz="0.0 0.0 0.0" rpy="0.0 0.0 0.0" />
+                <origin xyz="0.02 0.0 0.035" rpy="0.0 0.0 0.0" />
                 <geometry>
-                    <mesh filename="${mesh_url}astracamera.stl" scale="0.001 0.001 0.001" />
+                    <box size="0.04 0.15 0.03" />
+                    <!-- <mesh filename="${mesh_url}astracamera.stl" scale="0.001 0.001 0.001" /> -->
                 </geometry>
             </collision>

File: src/lidarino_description/urdf/lidarino_s2.urdf.xacro (robot description, xacro)
@@ -12,5 +12,7 @@
     <xacro:include filename="astra_camera.xacro" />
     <xacro:include filename="rplidars2.xacro" />
+    <xacro:include filename="imu.xacro" />
     <xacro:astra_camera parent="base_link" xyz="0.098 0.0 0.013" rpy="0 0 3.141592653589793" />
     <xacro:rplidars2 parent="base_link" xyz="-0.031 0.0 0.043" rpy="0 0 0" />
+    <xacro:imu_sensor parent="base_link" xyz="0.03 0.0 0.004" rpy="0 0 0" />
 </robot>

File: src/lidarino_description/urdf/rplidars2.xacro (robot description, xacro)
@@ -16,7 +16,8 @@
             </visual>
             <collision name="lidar_collision">
-                <origin xyz="0.0 0.0 0.0" rpy="0.0 0.0 0.0" />
+                <origin xyz="0.0 0.0 0.03" rpy="0.0 0.0 0.0" />
                 <geometry>
-                    <mesh filename="${mesh_url}RPLIDARS2.stl" scale="0.001 0.001 0.001" />
+                    <cylinder radius="0.035" length="0.02" />
+                    <!-- <mesh filename="${mesh_url}RPLIDARS2.stl" scale="0.001 0.001 0.001" /> -->
                 </geometry>
             </collision>
