Commit message: Chore: third-party ROS 2 packages added via .repos - Added m-explore-ros2 and sllidar_ros2 as third-party packages in the src directory. - Created lidarino_hardware package with necessary files and configurations. - lidarino_hardware package includes a custom hardware interface for Lidarino for communication between Orange Pi and ESP32. - Updated .gitignore - Updated README.md

File: src/lidarino_description/urdf/lidarino_ros2_control.xacro (robot description, xacro)
@@ -1,19 +1,28 @@
 <?xml version='1.0' encoding='utf-8'?>
 <robot xmlns:xacro="http://www.ros.org/wiki/xacro">
+    <xacro:arg name="use_sim" default="true" />
     <xacro:macro name="lidarino_ros2_control" params="use_lidar_control">
-        <ros2_control name="GazeboSystem" type="system">
-            <hardware>
-                <plugin>gz_ros2_control/GazeboSimSystem</plugin>
-            </hardware>
-            <xacro:if value="${use_lidar_control}">
-                <joint name="lidar_Revolute">
-                    <command_interface name="velocity">
-                        <param name="min">-100</param>
-                        <param name="max">100</param>
-                    </command_interface>
-                    <state_interface name="position"/>
-                    <state_interface name="velocity"/>
-                </joint>
+        <ros2_control name="LidarinoSystem" type="system">
+            <xacro:if value="${use_sim}">
+                <hardware>
+                    <plugin>gz_ros2_control/GazeboSimSystem</plugin>
+                </hardware>
+                <xacro:if value="${use_lidar_control}">
+                    <joint name="lidar_Revolute">
+                        <command_interface name="velocity">
+                            <param name="min">-100</param>
+                            <param name="max">100</param>
+                        </command_interface>
+                        <state_interface name="position"/>
+                        <state_interface name="velocity"/>
+                    </joint>
+                </xacro:if>
             </xacro:if>
+            <xacro:unless value="${use_sim}">
+                <hardware>
+                    <plugin>lidarino_hardware/LidarinoSystemHardware</plugin>
+                    <param name="serial_port">/dev/ttyUSB0</param>
+                </hardware>
+            </xacro:unless>
             <joint name="R_wheel_Revolute">
                 <command_interface name="velocity">
