Commit message: Docker Compatibility and bug fixes

File: src/lidarino_description/urdf/lidarino_ros2_control.xacro (robot description, xacro)
@@ -2,5 +2,5 @@
 <robot xmlns:xacro="http://www.ros.org/wiki/xacro">
     <xacro:arg name="use_sim" default="true" />
-    <xacro:macro name="lidarino_ros2_control" params="use_lidar_control">
+    <xacro:macro name="lidarino_ros2_control" params="use_lidar_control use_sim">
         <ros2_control name="LidarinoSystem" type="system">
             <xacro:if value="${use_sim}">
@@ -22,5 +22,5 @@
                 <hardware>
                     <plugin>lidarino_hardware/LidarinoSystemHardware</plugin>
-                    <param name="serial_port">/dev/ttyUSB0</param>
+                    <param name="serial_port">/dev/ttyACM0</param>
                 </hardware>
             </xacro:unless>

File: src/lidarino_description/urdf/lidarino_s2.urdf.xacro (robot description, xacro)
@@ -10,5 +10,5 @@
     <xacro:include filename="lidarino_ros2_control.xacro" />
     <xacro:lidarino_gazebo yaml_file="$(arg yaml_file)" />
-    <xacro:lidarino_ros2_control use_lidar_control="${use_lidar_control}" use_sim="${use_sim}" />
+    <xacro:lidarino_ros2_control use_lidar_control="${use_lidar_control}" use_sim="$(arg use_sim)" />
     <xacro:include filename="astra_camera.xacro" />
     <xacro:include filename="rplidars2.xacro" />
