Commit message: Bug fix and odom - Now ros_manager.py is working on Windows. - Added file .usda to lfs tracking. - Added damping and friction to the wheels in the URDF file. - Now StageIsaac.usd is publishing clock, odom and tf topics.

File: src/lidarino_description/urdf/lidarino_core_s2.xacro (robot description, xacro)
@@ -107,4 +107,5 @@
         <axis xyz="0.0 0.0 -1.0" />
         <limit effort="10.0" velocity="20.0" />
+        <dynamics damping="10000000.0" friction="0.1" />
     </joint>
     <joint name="R_wheel_Revolute" type="continuous">
@@ -114,4 +115,5 @@
         <axis xyz="0.0 0.0 1.0" />
         <limit effort="10.0" velocity="20.0" />
+        <dynamics damping="10000000.0" friction="0.1" />
     </joint>
     <joint name="caster_fixed" type="fixed">
