Commit message: Updated mesh files and URDF - Updated all the mesh file with the new mesh files from the CAD model. - Updated the URDF files to reflect the new mesh files, their positions and the collision geometry. - Moved the position of the IMU to the correct position in the URDF. - Updated the USD files to reflect the new mesh files and their positions. - Updated README.md. - Added fixed link/joint for the lid of the robot.

File: src/lidarino_description/urdf/imu.xacro (robot description, xacro)
@@ -18,5 +18,5 @@
                 <origin xyz="0 0 0" rpy="0 0 0" />
                 <geometry>
-                    <box size="0.02 0.02 0.005" />
+                    <box size="0.005 0.005 0.005" />
                 </geometry>
                 <material name="dark_grey" />
@@ -25,5 +25,5 @@
                 <origin xyz="0 0 0" rpy="0 0 0" />
                 <geometry>
-                    <box size="0.02 0.02 0.005" />
+                    <box size="0.005 0.005 0.005" />
                 </geometry>
             </collision>

File: src/lidarino_description/urdf/isaac.urdf (robot description, URDF)
Before this commit: robot lidarino, 9 links, 8 joints
Links:
- added link body_lid, mass 0.05261379951215123; collision box size=0.206 0.164 0.014; visual mesh filename=package://lidarino_description/urdf/meshes/bodyLid.stl scale=0.001 0.001 0.001
- link base_link: mass 0.33360490904476603 -> 0.4239314641509377; geometry collision box size=0.25 0.16 0.042; visual mesh filename=package://lidarino_description/urdf/meshes/base_link_s2.stl scale=0.001 0.001 0.001
- link imu_link: geometry collision box size=0.005 0.005 0.005; visual box size=0.005 0.005 0.005
Joints:
- added joint body_lid_fixed: type fixed, parent base_link, child body_lid, origin xyz=0.0 0.0 0.07 rpy=0.0 0.0 0.0
- joint L_wheel_Revolute: origin xyz=-0.06 0.06 0.015 rpy=1.5707963267948966 -0.0 0.0 -> xyz=-0.085 0.06 0.015 rpy=1.5707963267948966 -0.0 0.0
- joint R_wheel_Revolute: origin xyz=-0.06 -0.06 0.015 rpy=-1.5707963267948966 -0.0 0.0 -> xyz=-0.085 -0.06 0.015 rpy=-1.5707963267948966 -0.0 0.0
- joint astra_joint: origin xyz=0.098 0.0 0.013 rpy=0 0 3.141592653589793 -> xyz=0.120 0.0 0.025 rpy=0 0 3.141592653589793
- joint caster_fixed: origin xyz=0.052 0.0 -0.013 rpy=0.0 0.0 0.0 -> xyz=0.077 0.0 -0.013 rpy=0.0 0.0 0.0
- joint imu_joint: origin xyz=0.03 0.0 0.004 rpy=0 0 0 -> xyz=-0.092 0.0 0.02 rpy=0 0 0
- joint rplidars2_joint: origin xyz=-0.031 0.0 0.043 rpy=0 0 0 -> xyz=-0.056 0.0 0.053 rpy=0 0 0

File: src/lidarino_description/urdf/lidarino_core_s2.xacro (robot description, xacro)
@@ -4,6 +4,6 @@
         <inertial>
             <origin xyz="-0.0062724127968771535 1.3799035175597654e-08 0.013070827636125267" rpy="0.0 0.0 0.0" />
-            <mass value="0.33360490904476603" />
-            <inertia ixx="0.0006347717188410793" iyy="0.0009043843267201054" izz="0.001435861690423606" ixy="1.476040485669221e-10" iyz="-4.135017315855046e-11" ixz="4.795544012819681e-05" />
+            <mass value="0.4239314641509377" />
+            <inertia ixx="0.0010482842137546186" iyy="0.0024338106744802982" izz="0.003184067568059869" ixy="-9.417101996162051e-05" iyz="-2.234993490616969e-06" ixz="0.0001129151524043299" />
         </inertial>
         <visual name="base_link_visual">
@@ -15,7 +15,27 @@
         </visual>
         <collision name="base_link_collision">
-            <origin xyz="0.0 0.0 0.015" rpy="0.0 0.0 0.0" />
+            <origin xyz="0.0 0.0 0.021" rpy="0.0 0.0 0.0" />
             <geometry>
-                <box size="0.2 0.12 0.03" />
+                <box size="0.25 0.16 0.042" />
+            </geometry>
+        </collision>
+    </link>
+    <link name="body_lid">
+        <inertial>
+            <origin xyz="-0.012951394456098867 -3.147938388524642e-07 0.06881041966340294" rpy="0.0 0.0 0.0" />
+            <mass value="0.05261379951215123" />
+            <inertia ixx="0.0001489352862801382" iyy="0.000229958819591738" izz="0.00037746798651689653" ixy="3.80132469862603e-10" iyz="3.2124298873716476e-11" ixz="-6.825968075725163e-07" />
+        </inertial>
+        <visual name="body_lid_visual">
+            <origin xyz="0.0 0.0 -0.07" rpy="0.0 0.0 0.0" />
+            <geometry>
+                <mesh filename="${mesh_url}bodyLid.stl" scale="0.001 0.001 0.001" />
+            </geometry>
+            <material name="steel_blue" />
+        </visual>
+        <collision name="body_lid_collision">
+            <origin xyz="-0.024 0.0 -0.005" rpy="0.0 0.0 0.0" />
+            <geometry>
+                <box size="0.206 0.164 0.014" />
             </geometry>
         </collision>
@@ -82,5 +102,5 @@
     </link>
     <joint name="L_wheel_Revolute" type="continuous">
-        <origin xyz="-0.06 0.06 0.015" rpy="1.5707963267948966 -0.0 0.0" />
+        <origin xyz="-0.085 0.06 0.015" rpy="1.5707963267948966 -0.0 0.0" />
         <parent link="base_link" />
         <child link="wheel_L" />
@@ -89,5 +109,5 @@
     </joint>
     <joint name="R_wheel_Revolute" type="continuous">
-        <origin xyz="-0.06 -0.06 0.015" rpy="-1.5707963267948966 -0.0 0.0" />
+        <origin xyz="-0.085 -0.06 0.015" rpy="-1.5707963267948966 -0.0 0.0" />
         <parent link="base_link" />
         <child link="wheel_R" />
@@ -96,7 +116,12 @@
     </joint>
     <joint name="caster_fixed" type="fixed">
-        <origin xyz="0.052 0.0 -0.013" rpy="0.0 0.0 0.0" />
+        <origin xyz="0.077 0.0 -0.013" rpy="0.0 0.0 0.0" />
         <parent link="base_link" />
         <child link="caster" />
     </joint>
+    <joint name="body_lid_fixed" type="fixed">
+        <origin xyz="0.0 0.0 0.07" rpy="0.0 0.0 0.0" />
+        <parent link="base_link" />
+        <child link="body_lid" />
+    </joint>
 </robot>

File: src/lidarino_description/urdf/lidarino_isaac.urdf.xacro (robot description, xacro)
@@ -13,7 +13,7 @@
     <xacro:include filename="astra_camera.xacro" />
     <xacro:include filename="imu.xacro" />
-    <xacro:astra_camera parent="base_link" xyz="0.098 0.0 0.013" rpy="0 0 3.141592653589793" />
-    <xacro:rplidars2 parent="base_link" xyz="-0.031 0.0 0.043" rpy="0 0 0" />
-    <xacro:imu_sensor parent="base_link" xyz="0.03 0.0 0.004" rpy="0 0 0" />
+    <xacro:astra_camera parent="base_link" xyz="0.120 0.0 0.025" rpy="0 0 3.141592653589793" />
+    <xacro:rplidars2 parent="base_link" xyz="-0.056 0.0 0.053" rpy="0 0 0" />
+    <xacro:imu_sensor parent="base_link" xyz="-0.092 0.0 0.02" rpy="0 0 0" />
     <!--
          =========================================================

Commit message: URDF improvements and Isaac Sim integration.

File: src/lidarino_description/urdf/imu.xacro (robot description, xacro)
@@ -14,5 +14,5 @@
                 <origin xyz="0 0 0" rpy="0 0 0" />
                 <mass value="0.01" />
-                <inertia ixx="1e-6" iyy="1e-6" izz="1e-6" ixy="0.0" iyz="0.0" ixz="0.0" />
+                <inertia ixx="1e-4" iyy="1e-4" izz="1e-4" ixy="0.0" iyz="0.0" ixz="0.0" />
             </inertial>
             <visual name="imu_visual">

File: src/lidarino_description/urdf/isaac.urdf (robot description, URDF)
Before this commit: robot lidarino, 10 links, 9 joints
Links:
- link wheel_L: geometry collision cylinder length=0.025 radius=0.035; visual mesh filename=package://lidarino_description/urdf/meshes/wheel_L.stl scale=0.001 0.001 0.001
- link wheel_R: geometry collision cylinder length=0.025 radius=0.035; visual mesh filename=package://lidarino_description/urdf/meshes/wheel_R.stl scale=0.001 0.001 0.001

File: src/lidarino_description/urdf/lidarino_core_s2.xacro (robot description, xacro)
@@ -45,5 +45,5 @@
             <origin xyz="0.0 0.0 0.0" rpy="0.0 0.0 0.0" />
             <mass value="0.01" />
-            <inertia ixx="1e-6" iyy="1e-6" izz="1e-6" ixy="0" iyz="0" ixz="0" />
+            <inertia ixx="1e-4" iyy="1e-4" izz="1e-4" ixy="0" iyz="0" ixz="0" />
         </inertial>
         <visual name="caster_visual">
@@ -77,5 +77,5 @@
             <origin xyz="0 0 -0.017" rpy="0 0 0" />
             <geometry>
-                <sphere radius="0.035" />
+                <cylinder radius="0.035" length="0.025" />
             </geometry>
         </collision>
@@ -97,5 +97,5 @@
             <origin xyz="0 0 -0.017" rpy="0 0 0" />
             <geometry>
-                <sphere radius="0.035" />
+                <cylinder radius="0.035" length="0.025" />
             </geometry>
         </collision>
@@ -106,5 +106,5 @@
         <child link="wheel_L" />
         <axis xyz="0.0 0.0 -1.0" />
-        <limit effort="10.0" velocity="20.0" />
+        <limit effort="1000.0" velocity="200.0" />
         <dynamics damping="10000000.0" friction="0.1" />
     </joint>
@@ -114,5 +114,5 @@
         <child link="wheel_R" />
         <axis xyz="0.0 0.0 1.0" />
-        <limit effort="10.0" velocity="20.0" />
+        <limit effort="1000.0" velocity="200.0" />
         <dynamics damping="10000000.0" friction="0.1" />
     </joint>

File: src/lidarino_description/urdf/lidarino_isaac.urdf.xacro (robot description, xacro)
@@ -14,5 +14,5 @@
     <xacro:include filename="astra_camera.xacro" />
     <xacro:include filename="imu.xacro" />
-    <xacro:astra_camera parent="base_link" xyz="0.120 0.0 0.025" rpy="0 0 3.141592653589793" />
+    <xacro:astra_camera parent="base_link" xyz="0.120 0.0 0.025" rpy="1.570796 -1.570796 0" />
     <xacro:rplidars2 parent="base_link" xyz="-0.056 0.0 0.053" rpy="0 0 0" />
     <xacro:imu_sensor parent="base_link" xyz="-0.092 0.0 0.02" rpy="0 0 0" />
